Commit message: Fix constraint projector

File: assets/urdf/objects/cube_multicolor_allegro.urdf (robot description, URDF)
Before this commit: robot object, 1 links, 0 joints
Links:
- link object: mass None -> 0.5

File: assets/urdf/tip.urdf (robot description, URDF)
Before this commit: robot aux1, 4 links, 3 joints
Links:
- link ball: geometry collision sphere radius=0.008; visual sphere radius=0.01

Commit message: add friction support debug constraint projector

File: assets/urdf/objects/cube_multicolor_allegro.urdf (robot description, URDF)
Before this commit: robot object, 1 links, 0 joints
Links:
- link object: mass 0.5 -> None
