Commit message: Add GPT generated code for revised action space

File: assets/urdf/tip.urdf (robot description, URDF)
Before this commit: robot aux1, 4 links, 3 joints
Links:
- link ball: geometry collision sphere radius=0.01; visual sphere radius=0.01
Joints:
- joint aux1_ball: limit lower=-20.0 upper=20.0 effort=100 velocity=3.0 -> lower=0.0 upper=0.6 effort=100 velocity=3.0; origin xyz=0 0 1 rpy=0 0 0 -> xyz=0 0 0 rpy=0 0 0
- joint aux_aux1: limit lower=-20.0 upper=20.0 effort=100 velocity=3.0 -> lower=-0.3 upper=0.3 effort=100 velocity=3.0; origin xyz=0 0 1 rpy=0 0 0 -> xyz=0 0 0 rpy=0 0 0
- joint root_aux: limit lower=-20.0 upper=20.0 effort=100 velocity=3.0 -> lower=-0.3 upper=0.3 effort=100 velocity=3.0; origin xyz=0 0 1 rpy=0 0 0 -> xyz=0 0 0 rpy=0 0 0

Commit message: add detachment prevention projector

File: assets/urdf/tip.urdf (robot description, URDF)
Before this commit: robot aux1, 4 links, 3 joints
Joints:
- joint aux1_ball: axis 0 0 1 -> 0 0 -1

Commit message: keep debugging and add interpolation for target reaching

File: assets/urdf/tip.urdf (robot description, URDF)
Before this commit: robot aux1, 4 links, 3 joints
Joints:
- joint aux1_ball: limit lower=0.0 upper=0.6 effort=100 velocity=3.0 -> lower=0.0 upper=0.2 effort=100 velocity=3.0
- joint aux_aux1: limit lower=-0.3 upper=0.3 effort=100 velocity=3.0 -> lower=-0.15 upper=0.15 effort=100 velocity=3.0
- joint root_aux: limit lower=-0.3 upper=0.3 effort=100 velocity=3.0 -> lower=-0.15 upper=0.15 effort=100 velocity=3.0

Commit message: Fix reset bug

File: assets/urdf/tip.urdf (robot description, URDF)
Before this commit: robot aux1, 4 links, 3 joints
Joints:
- joint aux_aux1: limit lower=-0.15 upper=0.15 effort=100 velocity=3.0 -> lower=-0.08 upper=0.08 effort=100 velocity=3.0
- joint root_aux: limit lower=-0.15 upper=0.15 effort=100 velocity=3.0 -> lower=-0.08 upper=0.08 effort=100 velocity=3.0

Commit message: Add GPIS and grasp verifier

File: assets/urdf/tip.urdf (robot description, URDF)
Before this commit: robot aux1, 4 links, 3 joints
Joints:
- joint aux1_ball: axis 0 0 -1 -> 0 0 1; limit lower=0.0 upper=0.2 effort=100 velocity=3.0 -> lower=0.07 upper=0.13 effort=100 velocity=3.0
