Commit message: Enable full hand grasp

File: isaacgymenvs/grasping/pybullet_robot/src/pybullet_robot/robots/leap_hand/assets/leap_hand/robot.urdf (robot description, URDF)
Before this commit: robot onshape, 17 links, 16 joints
Links:
- link fingertip: geometry collision mesh filename=fingertip_round.stl; visual mesh filename=fingertip_round.stl
- link fingertip_2: geometry collision mesh filename=fingertip_round.stl; visual mesh filename=fingertip_round.stl
- link fingertip_3: geometry collision mesh filename=fingertip_round.stl; visual mesh filename=fingertip_round.stl
- link thumb_fingertip: geometry collision mesh filename=thumb_fingertip_round.stl; visual mesh filename=thumb_fingertip_round.stl
