Commit message: Add banana experiment

File: isaacgymenvs/grasping/assets/banana/banana.urdf (robot description, URDF)
Before this commit: robot banana, 1 links, 0 joints
Links:
- link banana: geometry collision mesh filename=decomp_textured.obj scale=1 1 1; visual mesh filename=textured.obj scale=1 1 1

File: isaacgymenvs/grasping/assets/hammer/hammer.urdf (robot description, URDF)
Before this commit: robot object, 1 links, 0 joints
Links:
- link object: mass 0.1 -> 0.05; geometry collision cylinder length=0.3 radius=0.015; visual mesh filename=textured.stl scale=1 1 1

Commit message: stable grasping with joint optimization

File: isaacgymenvs/grasping/assets/banana/banana.urdf (robot description, URDF)
Before this commit: robot banana, 1 links, 0 joints
Links:
- link banana: geometry collision mesh filename=textured_decomp.obj scale=1 1 1; visual mesh filename=textured_decomp.obj scale=1 1 1
