Commit message: add experiment scripts

File: assets/banana/banana.urdf (robot description, URDF)
Before this commit: robot banana, 1 links, 0 joints
Links:
- link banana: geometry collision mesh filename=banana_decomp.obj scale=1 1 1; visual mesh filename=banana.obj scale=1 1 1

File: assets/hammer/hammer.urdf (robot description, URDF)
Before this commit: robot object, 1 links, 0 joints
Links:
- link object: geometry collision mesh filename=hammer_decomp.obj scale=1 1 1; visual mesh filename=hammer.obj scale=1 1 1

File: assets/lego/lego.urdf (robot description, URDF)
Before this commit: robot object, 1 links, 0 joints
Links:
- link object: geometry collision mesh filename=lego_decomp.obj scale=1 1 1; visual mesh filename=lego.obj scale=1 1 1

File: assets/mug/mug.urdf (robot description, URDF)
Before this commit: robot object, 1 links, 0 joints
Links:
- link object: geometry collision mesh filename=mug_decomp.obj scale=1 1 1; visual mesh filename=mug.obj scale=1 1 1

File: assets/mug2/mug2.urdf (robot description, URDF)
Before this commit: robot object, 1 links, 0 joints
Links:
- link object: geometry collision mesh filename=mug2_decomp.obj scale=1 1 1; visual mesh filename=mug2.obj scale=1 1 1
