Commit message: add arm hand system optimization

File: pybullet_robot/src/pybullet_robot/robots/allegro_hand/models/allegro_hand_description_right.urdf (robot description, URDF)
Before this commit: robot allegro_hand_right, 22 links, 21 joints
Links:
- link hand_root: mass None -> 0.1
Joints:
- joint root_to_base: origin xyz=0 0 0 rpy=0 1.571 -1.571 -> xyz=0 0 0 rpy=0 1.571 0
