Commit message: add changes to real robot experiment

File: assets/kuka_allegro/model.urdf (robot description, URDF)
Before this commit: robot lbr_iiwa, 30 links, 29 joints
Links:
- removed link link_0.0
- removed link link_1.0
- removed link link_10.0
- removed link link_11.0
- removed link link_11.0_tip
- removed link link_12.0
- removed link link_13.0
- removed link link_14.0
- removed link link_15.0
- removed link link_15.0_tip
- removed link link_2.0
- removed link link_3.0
- removed link link_3.0_tip
- removed link link_4.0
- removed link link_5.0
- removed link link_6.0
- removed link link_7.0
- removed link link_7.0_tip
- removed link link_8.0
- removed link link_9.0
Joints:
- removed joint joint_0.0
- removed joint joint_1.0
- removed joint joint_10.0
- removed joint joint_11.0
- removed joint joint_11.0_tip
- removed joint joint_12.0
- removed joint joint_13.0
- removed joint joint_14.0
- removed joint joint_15.0
- removed joint joint_15.0_tip
- removed joint joint_2.0
- removed joint joint_3.0
- removed joint joint_3.0_tip
- removed joint joint_4.0
- removed joint joint_5.0
- removed joint joint_6.0
- removed joint joint_7.0
- removed joint joint_7.0_tip
- removed joint joint_8.0
- removed joint joint_9.0
- joint lbr_iiwa_joint_7: origin xyz=0 0.081 0 rpy=-1.57079632679 3.14159265359 0 -> xyz=0 0.081 0 rpy=-1.57079632679 3.9269908169872414 0.0

Commit message: synchronize

File: assets/kuka_allegro/model.urdf (robot description, URDF)
Before this commit: robot lbr_iiwa, 10 links, 9 joints
Joints:
- joint lbr_iiwa_joint_1: limit lower=-2.96705972839 upper=2.96705972839 effort=300 velocity=10 -> lower=-2.85 upper=2.85 effort=300 velocity=10
- joint lbr_iiwa_joint_2: limit lower=-2.09439510239 upper=2.09439510239 effort=300 velocity=10 -> lower=-2.0 upper=2.0 effort=300 velocity=10
- joint lbr_iiwa_joint_3: limit lower=-2.96705972839 upper=2.96705972839 effort=300 velocity=10 -> lower=-2.85 upper=2.85 effort=300 velocity=10
- joint lbr_iiwa_joint_4: limit lower=-2.09439510239 upper=2.09439510239 effort=300 velocity=10 -> lower=-2.0 upper=2.0 effort=300 velocity=10
- joint lbr_iiwa_joint_5: limit lower=-2.96705972839 upper=2.96705972839 effort=300 velocity=10 -> lower=-2.85 upper=2.85 effort=300 velocity=10
- joint lbr_iiwa_joint_6: limit lower=-2.09439510239 upper=2.09439510239 effort=300 velocity=10 -> lower=-2.0 upper=2.0 effort=300 velocity=10
- joint lbr_iiwa_joint_7: limit lower=-3.05432619099 upper=3.05432619099 effort=300 velocity=10 -> lower=-3.0 upper=3.0 effort=300 velocity=10
